File: SandsOfTimePCB/SandsOfTimePCB/SandsOfTimePCB.kicad_pcb (KiCad board)
At the start: 2 copper layers, 8 parts, among them U1 DS3231M

Commit message: added files from old project
Parts:
- removed J_hbridge1_left1, J_hbridge1_right1, J_hbridge2_left1, J_hbridge2_right1, J_hbridge3_left1, J_hbridge3_right1: Conn_01x06_Female, Connector_PinSocket_2.54mm:PinSocket_1x06_P2.54mm_Vertical
- added Uhbridge1: DRV8801RTY, Connector_PinSocket_2.54mm:PinSocket_2x06_P2.54mm_Vertical, F.Cu at (205.7, 55.9)
- added Uhbridge2: DRV8801RTY, Connector_PinSocket_2.54mm:PinSocket_2x06_P2.54mm_Vertical, F.Cu at (199.4, 55.9)
- added Uhbridge3: DRV8801RTY, Connector_PinSocket_2.54mm:PinSocket_2x06_P2.54mm_Vertical, F.Cu at (172.7, 71.1)
- renumbered U1 to Utimer_chip1
