File: SandsOfTimePCB/SandsOfTimePCB/SandsOfTimePCB.kicad_sch (KiCad schematic)
At the start: 5 parts

Commit message: added files from old project
Parts:
- added J_encoder_pins1: Conn_02x15_Top_Bottom_MountingPin, symbol Connector_Generic_MountingPin:Conn_02x15_Top_Bottom_MountingPin
- Uhbridge1, Uhbridge2, Uhbridge3: footprint Package_DFN_QFN:Texas_S-PWQFN-N16_EP2.1x2.1mm_ThermalVias -> Connector_PinSocket_2.54mm:PinSocket_2x06_P2.54mm_Vertical
- renumbered Utimer_chip to Utimer_chip1
Changed lines of the file:
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@@
     (property "Reference" "Uhbridge3" (id 0) (at 231.14 123.19 0))
     (property "Value" "DRV8801RTY" (id 1) (at 231.14 125.73 0))
-    (property "Footprint" "Package_DFN_QFN:Texas_S-PWQFN-N16_EP2.1x2.1mm_ThermalVias" (id 2) (at 260.35 127 0)
+    (property "Footprint" "Connector_PinSocket_2.54mm:PinSocket_2x06_P2.54mm_Vertical" (id 2) (at 260.35 127 0)
       (effects (font (size 1.27 1.27)) hide)
     )
@@
     (property "Reference" "Uhbridge2" (id 0) (at 231.14 81.28 0))
     (property "Value" "DRV8801RTY" (id 1) (at 231.14 83.82 0))
-    (property "Footprint" "Package_DFN_QFN:Texas_S-PWQFN-N16_EP2.1x2.1mm_ThermalVias" (id 2) (at 260.35 85.09 0)
+    (property "Footprint" "Connector_PinSocket_2.54mm:PinSocket_2x06_P2.54mm_Vertical" (id 2) (at 260.35 85.09 0)
       (effects (font (size 1.27 1.27)) hide)
     )
@@
   (symbol (lib_id "Timer_RTC:DS3231M") (at 124.46 104.14 0) (unit 1)
     (in_bom yes) (on_board yes) (fields_autoplaced)
-    (property "Reference" "Utimer_chip" (id 0) (at 126.4794 114.3 0)
+    (property "Reference" "Utimer_chip1" (id 0) (at 126.4794 114.3 0)
       (effects (font (size 1.27 1.27)) (justify left))
     )
@@
     (property "Reference" "Uhbridge1" (id 0) (at 231.14 36.83 0))
     (property "Value" "DRV8801RTY" (id 1) (at 231.14 39.37 0))
-    (property "Footprint" "Package_DFN_QFN:Texas_S-PWQFN-N16_EP2.1x2.1mm_ThermalVias" (id 2) (at 260.35 40.64 0)
+    (property "Footprint" "Connector_PinSocket_2.54mm:PinSocket_2x06_P2.54mm_Vertical" (id 2) (at 260.35 40.64 0)
       (effects (font (size 1.27 1.27)) hide)
     )
@@
     (pin "8")
     (pin "9")
+  )
+  (symbol (lib_id "Connector_Generic_MountingPin:Conn_02x15_Top_Bottom_MountingPin") (at 119.38 54.61 0) (unit 1)
+    (in_bom yes) (on_board yes) (fields_autoplaced)
+    (property "Reference" "J_encoder_pins1" (id 0) (at 120.65 30.48 0))
+    (property "Value" "Conn_02x15_Top_Bottom_MountingPin" (id 1) (at 120.65 33.02 0))
+    (property "Footprint" "" (id 2) (at 119.38 54.61 0)
+      (effects (font (size 1.27 1.27)) hide)
+    )
+    (property "Datasheet" "~" (id 3) (at 119.38 54.61 0)
+      (effects (font (size 1.27 1.27)) hide)
+    )
+    (pin "1")
+    (pin "10")
+    (pin "11")
+    (pin "12")
+    (pin "13")
+    (pin "14")
+    (pin "15")
+    (pin "16")
+    (pin "17")
+    (pin "18")
+    (pin "19")
+    (pin "2")
+    (pin "20")
+    (pin "21")
+    (pin "22")
+    (pin "23")
+    (pin "24")
+    (pin "25")
+    (pin "26")
+    (pin "27")
+    (pin "28")
+    (pin "29")
+    (pin "3")
+    (pin "30")
+    (pin "4")
+    (pin "5")
+    (pin "6")
+    (pin "7")
+    (pin "8")
+    (pin "9")
+    (pin "MP")
   )
   (symbol (lib_id "Comparator:MAX941xPA") (at 162.56 127 0) (unit 1)
@@
   )
   (symbol_instances
+    (path "/e8713bbb-a454-4ab0-bcce-b334146330b5"
+      (reference "J_encoder_pins1") (unit 1) (value "Conn_02x15_Top_Bottom_MountingPin") (footprint "")
+    )
     (path "/fc2c05ae-aae7-4fcc-bfac-80ece148f9ac"
       (reference "Ucomparator1") (unit 1) (value "MAX941xPA") (footprint "Package_DIP:DIP-8_W7.62mm_Socket")
     )
     (path "/bec2044d-658d-4d80-9e0b-b6645a10363e"
-      (reference "Uhbridge1") (unit 1) (value "DRV8801RTY") (footprint "Package_DFN_QFN:Texas_S-PWQFN-N16_EP2.1x2.1mm_ThermalVias")
+      (reference "Uhbridge1") (unit 1) (value "DRV8801RTY") (footprint "Connector_PinSocket_2.54mm:PinSocket_2x06_P2.54mm_Vertical")
     )
     (path "/685aa86d-2ed0-4abc-82c2-1e7183ab195a"
-      (reference "Uhbridge2") (unit 1) (value "DRV8801RTY") (footprint "Package_DFN_QFN:Texas_S-PWQFN-N16_EP2.1x2.1mm_ThermalVias")
+      (reference "Uhbridge2") (unit 1) (value "DRV8801RTY") (footprint "Connector_PinSocket_2.54mm:PinSocket_2x06_P2.54mm_Vertical")
     )
     (path "/639c8661-7489-4420-bca8-db8d3729e1b4"
-      (reference "Uhbridge3") (unit 1) (value "DRV8801RTY") (footprint "Package_DFN_QFN:Texas_S-PWQFN-N16_EP2.1x2.1mm_ThermalVias")
+      (reference "Uhbridge3") (unit 1) (value "DRV8801RTY") (footprint "Connector_PinSocket_2.54mm:PinSocket_2x06_P2.54mm_Vertical")
     )
     (path "/8e9849a5-8cfa-4079-a4fe-fefea44e2f0e"
-      (reference "Utimer_chip") (unit 1) (value "DS3231M") (footprint "Connector_PinSocket_2.54mm:PinSocket_1x07_P2.54mm_Vertical")
+      (reference "Utimer_chip1") (unit 1) (value "DS3231M") (footprint "Connector_PinSocket_2.54mm:PinSocket_1x07_P2.54mm_Vertical")
     )
   )
